File: Sauna.kicad_pcb (KiCad board)
At the start: 2 copper layers, 7 parts, among them J1 Barrel_Jack_MountingPin, J2 Screw_Terminal_01x02, J3 Screw_Terminal_01x03, K1 FINDER-40.11, Q1 2N2219, U1 NodeMCU_1.0_(ESP-12E)

Commit message: ver 0.11
Routing:
- net GND: track 164.5 -> 156.7 mm
- net +10V: track 87.3 -> 89.9 mm
- net Net-(J2-Pad1): track 32.5 -> 31.2 mm
- added copper zone on F.Cu, net (none)
Changed lines of the file:
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@@
     (thickness 1.6)
     (drawings 0)
-    (tracks 39)
+    (tracks 42)
     (zones 0)
     (modules 7)
@@
     (solder_mask_min_width 0.25)
     (aux_axis_origin 0 0)
-    (visible_elements FFFFFF7F)
+    (visible_elements 7FFFFFFF)
     (pcbplotparams
       (layerselection 0x010fc_ffffffff)
@@
   )
   (segment (start 96.52 72.39) (end 96.52 70.39) (width 0.25) (layer F.Cu) (net 1))
-  (segment (start 96.52 72.39) (end 106.68 72.39) (width 0.25) (layer F.Cu) (net 1))
-  (segment (start 138.43 97.79) (end 132.08 97.79) (width 0.25) (layer F.Cu) (net 1))
-  (segment (start 132.08 97.79) (end 106.68 72.39) (width 0.25) (layer F.Cu) (net 1))
-  (segment (start 106.68 72.39) (end 106.68 64.77) (width 0.25) (layer F.Cu) (net 1))
-  (segment (start 106.68 64.77) (end 115.57 55.88) (width 0.25) (layer F.Cu) (net 1))
-  (segment (start 115.57 55.88) (end 189.23 55.88) (width 0.25) (layer F.Cu) (net 1))
   (segment (start 189.23 66.66) (end 193.04 70.47) (width 0.25) (layer F.Cu) (net 1))
-  (segment (start 189.23 55.88) (end 189.23 66.66) (width 0.25) (layer F.Cu) (net 1))
-  (segment (start 87.63 81.28) (end 106.68 100.33) (width 0.25) (layer F.Cu) (net 2))
-  (segment (start 87.63 73.68) (end 87.63 81.28) (width 0.25) (layer F.Cu) (net 2))
-  (segment (start 90.52 72.39) (end 88.92 72.39) (width 0.25) (layer F.Cu) (net 2))
-  (segment (start 88.92 72.39) (end 87.63 73.68) (width 0.25) (layer F.Cu) (net 2))
-  (segment (start 132.08 117.89) (end 132.08 100.33) (width 0.25) (layer F.Cu) (net 2))
-  (segment (start 106.68 100.33) (end 132.08 100.33) (width 0.25) (layer F.Cu) (net 2))
+  (segment (start 96.52 72.39) (end 125.73 72.39) (width 1) (layer F.Cu) (net 1))
+  (segment (start 125.73 72.39) (end 125.73 64.77) (width 1) (layer F.Cu) (net 1))
+  (segment (start 125.73 64.77) (end 135.89 54.61) (width 1) (layer F.Cu) (net 1))
+  (segment (start 177.18 54.61) (end 193.04 70.47) (width 1) (layer F.Cu) (net 1))
+  (segment (start 135.89 54.61) (end 177.18 54.61) (width 1) (layer F.Cu) (net 1))
+  (segment (start 125.73 72.39) (end 125.73 91.44) (width 0.25) (layer F.Cu) (net 1))
+  (segment (start 125.73 91.44) (end 132.08 97.79) (width 0.25) (layer F.Cu) (net 1))
+  (segment (start 132.08 97.79) (end 138.43 97.79) (width 0.25) (layer F.Cu) (net 1))
   (segment (start 132.08 100.33) (end 138.43 100.33) (width 0.25) (layer F.Cu) (net 2))
-  (segment (start 111.55 121.92) (end 115.58 117.89) (width 0.25) (layer F.Cu) (net 3))
-  (segment (start 109.22 121.92) (end 111.55 121.92) (width 0.25) (layer F.Cu) (net 3))
-  (segment (start 86.36 125.73) (end 105.41 125.73) (width 0.25) (layer F.Cu) (net 3))
-  (segment (start 105.41 125.73) (end 109.22 121.92) (width 0.25) (layer F.Cu) (net 3))
-  (segment (start 108.24 129.23) (end 112.08 125.39) (width 0.25) (layer F.Cu) (net 4))
-  (segment (start 86.36 129.23) (end 108.24 129.23) (width 0.25) (layer F.Cu) (net 4))
+  (segment (start 88.92 72.39) (end 86.36 74.95) (width 1) (layer F.Cu) (net 2))
+  (segment (start 90.52 72.39) (end 88.92 72.39) (width 1) (layer F.Cu) (net 2))
+  (segment (start 86.36 74.95) (end 86.36 78.74) (width 1) (layer F.Cu) (net 2))
+  (segment (start 86.36 78.74) (end 116.84 109.22) (width 1) (layer F.Cu) (net 2))
+  (segment (start 123.41 109.22) (end 132.08 117.89) (width 1) (layer F.Cu) (net 2))
+  (segment (start 116.84 109.22) (end 123.41 109.22) (width 1) (layer F.Cu) (net 2))
+  (segment (start 132.08 100.33) (end 123.19 109.22) (width 0.25) (layer F.Cu) (net 2))
+  (segment (start 113.45868 117.89) (end 109.42868 121.92) (width 1) (layer F.Cu) (net 3))
+  (segment (start 115.58 117.89) (end 113.45868 117.89) (width 1) (layer F.Cu) (net 3))
+  (segment (start 109.42868 121.92) (end 91.44 121.92) (width 1) (layer F.Cu) (net 3))
+  (segment (start 91.44 121.92) (end 87.63 125.73) (width 1) (layer F.Cu) (net 3))
+  (segment (start 110.580001 126.889999) (end 112.08 125.39) (width 1) (layer F.Cu) (net 4))
+  (segment (start 108.24 129.23) (end 110.580001 126.889999) (width 1) (layer F.Cu) (net 4))
+  (segment (start 86.36 129.23) (end 108.24 129.23) (width 1) (layer F.Cu) (net 4))
   (segment (start 177.405 76.2) (end 177.8 75.805) (width 0.25) (layer F.Cu) (net 5))
   (segment (start 176.135 77.47) (end 177.8 75.805) (width 0.25) (layer F.Cu) (net 5))
@@
   (segment (start 161.29 110.49) (end 180.34 129.54) (width 0.25) (layer F.Cu) (net 7))
   (segment (start 161.29 76.2) (end 161.29 110.49) (width 0.25) (layer F.Cu) (net 7))
-  (segment (start 173.99 135.89) (end 177.8 132.08) (width 0.25) (layer F.Cu) (net 31))
-  (segment (start 132.08 135.89) (end 173.99 135.89) (width 0.25) (layer F.Cu) (net 31))
+  (segment (start 132.08 135.89) (end 173.99 135.89) (width 1) (layer F.Cu) (net 31))
+  (segment (start 173.99 135.89) (end 177.8 132.08) (width 1) (layer F.Cu) (net 31))
   (segment (start 166.37 80.01) (end 167.64 80.01) (width 0.25) (layer F.Cu) (net 34))
   (segment (start 167.64 80.01) (end 182.88 95.25) (width 0.25) (layer F.Cu) (net 34))
   (segment (start 182.88 95.25) (end 182.88 132.08) (width 0.25) (layer F.Cu) (net 34))
+  (zone (net 0) (net_name "") (layer F.Cu) (hatch edge 0.508)
+    (connect_pads (clearance 0.508))
+    (min_thickness 0.254)
+    (fill yes (arc_segments 16) (thermal_gap 0.508) (thermal_bridge_width 0.508))
+    (polygon
+      (pts
+        (xy 82.55 81.28) (xy 82.55 118.11) (xy 102.87 118.11) (xy 102.87 101.6)
+      )
+    )
+  )
+  (zone (net 0) (net_name "") (layer F.Cu) (hatch none 0.508)
+    (connect_pads (clearance 0.508))
+    (min_thickness 0.254)
+    (fill yes (arc_segments 16) (thermal_gap 0.508) (thermal_bridge_width 0.508) (smoothing chamfer))
+    (polygon
+      (pts
+        (xy 139.7 114.3) (xy 161.29 114.3) (xy 170.18 123.19) (xy 170.18 132.08) (xy 139.7 132.08)
+        (xy 139.7 120.65)
+      )
+    )
+  )
+  (zone (net 0) (net_name "") (layer F.Cu) (hatch none 0.508)
+    (connect_pads (clearance 0.508))
+    (min_thickness 0.254)
+    (fill yes (arc_segments 16) (thermal_gap 0.508) (thermal_bridge_width 0.508) (smoothing chamfer))
+    (polygon
+      (pts
+        (xy 83.82 53.34) (xy 132.08 53.34) (xy 118.11 67.31) (xy 83.82 66.04)
+      )
+    )
+  )
+  (zone (net 0) (net_name "") (layer F.Cu) (hatch none 0.508)
+    (connect_pads (clearance 0.508))
+    (min_thickness 0.254)
+    (fill yes (arc_segments 16) (thermal_gap 0.508) (thermal_bridge_width 0.508) (smoothing chamfer))
+    (polygon
+      (pts
+        (xy 171.45 88.9) (xy 171.45 116.84) (xy 179.07 124.46) (xy 179.07 96.52)
+      )
+    )
+  )
+  (zone (net 0) (net_name "") (layer F.Cu) (hatch none 0.508)
+    (connect_pads (clearance 0.508))
+    (min_thickness 0.254)
+    (fill yes (arc_segments 16) (thermal_gap 0.508) (thermal_bridge_width 0.508) (smoothing chamfer))
+    (polygon
+      (pts
+        (xy 176.53 83.82) (xy 198.12 83.82) (xy 198.12 137.16) (xy 185.42 125.73) (xy 185.42 92.71)
+      )
+    )
+  )
+  (zone (net 0) (net_name "") (layer F.Cu) (hatch none 0.508)
+    (connect_pads (clearance 0.508))
+    (min_thickness 0.254)
+    (fill yes (arc_segments 16) (thermal_gap 0.508) (thermal_bridge_width 0.508) (smoothing chamfer))
+    (polygon
+      (pts
+        (xy 90.17 77.47) (xy 123.19 77.47) (xy 123.19 92.71) (xy 129.54 99.06) (xy 124.46 105.41)
+        (xy 116.84 105.41) (xy 110.49 99.06)
+      )
+    )
+  )
+  (zone (net 0) (net_name "") (layer F.Cu) (hatch none 0.508)
+    (connect_pads (clearance 0.508))
+    (min_thickness 0.254)
+    (fill yes (arc_segments 16) (thermal_gap 0.508) (thermal_bridge_width 0.508) (smoothing chamfer))
+    (polygon
+      (pts
+        (xy 129.54 66.04) (xy 129.54 90.17) (xy 134.62 95.25) (xy 134.62 60.96)
+      )
+    )
+  )
+  (zone (net 0) (net_name "") (layer F.Cu) (hatch none 0.508)
+    (connect_pads (clearance 0.508))
+    (min_thickness 0.254)
+    (fill yes (arc_segments 16) (thermal_gap 0.508) (thermal_bridge_width 0.508) (smoothing chamfer))
+    (polygon
+      (pts
+        (xy 180.34 53.34) (xy 199.39 53.34) (xy 199.39 63.5) (xy 190.5 63.5)
+      )
+    )
+  )
 )
